File: bike-light-board.kicad_pcb (KiCad board)
At the start: 2 copper layers, 40.2 x 69 mm, 64 parts, among them J1 S2B-PH-SM4-TB, J2 USB_B_Micro, J3 AVR-ISP-6, P1 WirePad, P2 WirePad, P3 WirePad, P4 WirePad, Q1 NCE2003, Q2 NCE2003, Q3 NCE2003, Q4 SMD0805-20, SW1 SW_Push, U1 BRCL4054CME, U2 SSP6206-33NR, U3 QMA7981, U4 ATtiny84A-MU, U5 M74VHC1GT08DFT2G

Commit message: remove old v1 files
Parts:
- renumbered C2 to C1, C7 to C10, C9 to C11, C11 to C12, C12 to C13, C19 to C14, C3 to C2, C1 to C3, C20 to C4, C4 to C5, C8 to C7, C10 to C8, C5 to C9, D8 to D1, D7 to D2, D1 to D3, D2 to D4, D3 to D5, D4 to D6, D5 to D7, D6 to D8, J2 to J1, J1 to J2, P4 to P1, P1 to P2, P2 to P3, P3 to P4, R2 to R1, R9 to R10, R8 to R11, R11 to R12, R12 to R13, R20 to R14, R6 to R15, R19 to R16, R10 to R17, R13 to R18, R14 to R19, R3 to R2, R15 to R20, R24 to R21, R16 to R22, R17 to R23, R18 to R24, R4 to R3, R1 to R4, R21 to R5, R22 to R6, R23 to R7, R5 to R8, R7 to R9, U3 to U2, U2 to U3

Commit message: update broken library
Parts:
- added G***: LOGO, bike-light-board:Logo_Lil_Light_Long, B.Cu at (168.3, 123.3)
Connections:
- D1 pad 3: Net-(D1-Pad3) -> (no net)
- D8 pad 2: Net-(D8-Pad2) -> (no net)
- J1 pad 4: Net-(J1-Pad4) -> (no net)
- U2 pad 10: Net-(U2-Pad10) -> (no net)
- U2 pad 11: Net-(U2-Pad11) -> (no net)
- U2 pad 4: Net-(U2-Pad4) -> (no net)
- U2 pad 6: Net-(U2-Pad6) -> (no net)
- U4 pad 10: Net-(U4-Pad10) -> (no net)
- U4 pad 17: Net-(U4-Pad17) -> (no net)
- U4 pad 18: Net-(U4-Pad18) -> (no net)
- U4 pad 19: Net-(U4-Pad19) -> (no net)
- U4 pad 6: Net-(U4-Pad6) -> (no net)
- U4 pad 7: Net-(U4-Pad7) -> (no net)
