File: bike-light-board.sch (KiCad schematic (older format))
At the start: 70 parts, among them J1 S2B-PH-SM4-TB, J2 USB_B_Micro, J3 AVR-ISP-6, P1 WirePad, P2 WirePad, P3 WirePad, P4 WirePad, Q1 NCE2003, Q2 NCE2003, Q3 NCE2003, Q4 SMD0805-20, SW1 SW_Push, U1 BRCL4054CME, U2 SSP6206-33NR, U3 QMA7981, U4 ATtiny84A-MU, U5 M74VHC1GT08DFT2G

Commit message: remove front led caps
Parts:
- removed C13, C14, C15, C16, C17, C18: 100n, Capacitor_SMD:C_0402_1005Metric, symbol Device:C
Changed lines of the file:
@@
 Wire Wire Line
 	12300 5600 12300 5850
-Connection ~ 12800 6000
 Wire Wire Line
 	12650 6150 12600 6150
@@
 	1    0    0    -1
 $EndComp
-$Comp
-L Device:C C18
-U 1 1 5E7BF3EB
-P 12800 6150
-F 0 "C18" H 12915 6196 50  0000 L CNN
-F 1 "100n" H 12915 6105 50  0000 L CNN
-F 2 "Capacitor_SMD:C_0402_1005Metric" H 12838 6000 50  0001 C CNN
-F 3 "~" H 12800 6150 50  0001 C CNN
-F 4 "C60474" H 12800 6150 50  0001 C CNN "LCSC Part Number"
-F 5 "" H 12800 6150 50  0001 C CNN "Voltage"
-	1    12800 6150
-	1    0    0    -1
-$EndComp
-$Comp
-L power:GND #PWR066
-U 1 1 5E7BF3E5
-P 12800 6300
-F 0 "#PWR066" H 12800 6050 50  0001 C CNN
-F 1 "GND" H 12805 6127 50  0000 C CNN
-F 2 "" H 12800 6300 50  0001 C CNN
-F 3 "" H 12800 6300 50  0001 C CNN
-	1    12800 6300
-	1    0    0    -1
-$EndComp
-Connection ~ 12800 5150
 Wire Wire Line
 	12800 5150 12650 5150
@@
 	1    0    0    -1
 $EndComp
-$Comp
-L Device:C C17
-U 1 1 5E7BF3CF
-P 12800 5300
-F 0 "C17" H 12915 5346 50  0000 L CNN
-F 1 "100n" H 12915 5255 50  0000 L CNN
-F 2 "Capacitor_SMD:C_0402_1005Metric" H 12838 5150 50  0001 C CNN
-F 3 "~" H 12800 5300 50  0001 C CNN
-F 4 "C60474" H 12800 5300 50  0001 C CNN "LCSC Part Number"
-F 5 "" H 12800 5300 50  0001 C CNN "Voltage"
-	1    12800 5300
-	1    0    0    -1
-$EndComp
-$Comp
-L power:GND #PWR064
-U 1 1 5E7BF3C9
-P 12800 5450
-F 0 "#PWR064" H 12800 5200 50  0001 C CNN
-F 1 "GND" H 12805 5277 50  0000 C CNN
-F 2 "" H 12800 5450 50  0001 C CNN
-F 3 "" H 12800 5450 50  0001 C CNN
-	1    12800 5450
-	1    0    0    -1
-$EndComp
 Wire Wire Line
 	12300 4750 12300 5000
 Wire Wire Line
 	12300 3900 12300 4150
-Connection ~ 12800 4300
 Wire Wire Line
 	12800 4300 12650 4300
@@
 	1    0    0    -1
 $EndComp
-$Comp
-L Device:C C16
-U 1 1 5E7B90DA
-P 12800 4450
-F 0 "C16" H 12915 4496 50  0000 L CNN
-F 1 "100n" H 12915 4405 50  0000 L CNN
-F 2 "Capacitor_SMD:C_0402_1005Metric" H 12838 4300 50  0001 C CNN
-F 3 "~" H 12800 4450 50  0001 C CNN
-F 4 "C60474" H 12800 4450 50  0001 C CNN "LCSC Part Number"
-F 5 "" H 12800 4450 50  0001 C CNN "Voltage"
-	1    12800 4450
-	1    0    0    -1
-$EndComp
-$Comp
-L power:GND #PWR062
-U 1 1 5E7B90D4
-P 12800 4600
-F 0 "#PWR062" H 12800 4350 50  0001 C CNN
-F 1 "GND" H 12805 4427 50  0000 C CNN
-F 2 "" H 12800 4600 50  0001 C CNN
-F 3 "" H 12800 4600 50  0001 C CNN
-	1    12800 4600
-	1    0    0    -1
-$EndComp
-Connection ~ 12800 3450
 Wire Wire Line
 	12650 3600 12600 3600
@@
 	1    0    0    -1
 $EndComp
-$Comp
-L Device:C C15
-U 1 1 5E7B90BE
-P 12800 3600
-F 0 "C15" H 12915 3646 50  0000 L CNN
-F 1 "100n" H 12915 3555 50  0000 L CNN
-F 2 "Capacitor_SMD:C_0402_1005Metric" H 12838 3450 50  0001 C CNN
-F 3 "~" H 12800 3600 50  0001 C CNN
-F 4 "C60474" H 12800 3600 50  0001 C CNN "LCSC Part Number"
-F 5 "" H 12800 3600 50  0001 C CNN "Voltage"
-	1    12800 3600
-	1    0    0    -1
-$EndComp
-$Comp
-L power:GND #PWR060
-U 1 1 5E7B90B8
-P 12800 3750
-F 0 "#PWR060" H 12800 3500 50  0001 C CNN
-F 1 "GND" H 12805 3577 50  0000 C CNN
-F 2 "" H 12800 3750 50  0001 C CNN
-F 3 "" H 12800 3750 50  0001 C CNN
-	1    12800 3750
-	1    0    0    -1
-$EndComp
 Wire Wire Line
 	12300 3050 12300 3300
 Wire Wire Line
 	12300 2200 12300 2450
-Connection ~ 12800 2600
 Wire Wire Line
 	12650 2750 12600 2750
@@
 	1    0    0    -1
 $EndComp
-$Comp
-L Device:C C14
-U 1 1 5E7A3139
-P 12800 2750
-F 0 "C14" H 12915 2796 50  0000 L CNN
-F 1 "100n" H 12915 2705 50  0000 L CNN
-F 2 "Capacitor_SMD:C_0402_1005Metric" H 12838 2600 50  0001 C CNN
-F 3 "~" H 12800 2750 50  0001 C CNN
-F 4 "C60474" H 12800 2750 50  0001 C CNN "LCSC Part Number"
-F 5 "" H 12800 2750 50  0001 C CNN "Voltage"
-	1    12800 2750
-	1    0    0    -1
-$EndComp
-$Comp
-L power:GND #PWR058
-U 1 1 5E7A3133
-P 12800 2900
-F 0 "#PWR058" H 12800 2650 50  0001 C CNN
-F 1 "GND" H 12805 2727 50  0000 C CNN
-F 2 "" H 12800 2900 50  0001 C CNN
-F 3 "" H 12800 2900 50  0001 C CNN
-	1    12800 2900
-	1    0    0    -1
-$EndComp
-Connection ~ 12800 1750
 Wire Wire Line
 	12650 1900 12600 1900
@@
 	1    0    0    -1
 $EndComp
-$Comp
-L Device:C C13
-U 1 1 5E737FBF
-P 12800 1900
-F 0 "C13" H 12915 1946 50  0000 L CNN
-F 1 "100n" H 12915 1855 50  0000 L CNN
-F 2 "Capacitor_SMD:C_0402_1005Metric" H 12838 1750 50  0001 C CNN
-F 3 "~" H 12800 1900 50  0001 C CNN
-F 4 "C60474" H 12800 1900 50  0001 C CNN "LCSC Part Number"
-F 5 "" H 12800 1900 50  0001 C CNN "Voltage"
-	1    12800 1900
-	1    0    0    -1
-$EndComp
-$Comp
-L power:GND #PWR056
-U 1 1 5E737FB9
-P 12800 2050
-F 0 "#PWR056" H 12800 1800 50  0001 C CNN
-F 1 "GND" H 12805 1877 50  0000 C CNN
-F 2 "" H 12800 2050 50  0001 C CNN
-F 3 "" H 12800 2050 50  0001 C CNN
-	1    12800 2050
-	1    0    0    -1
-$EndComp

Commit message: remove old v1 files
Parts:
- renumbered C2 to C1, C7 to C10, C9 to C11, C11 to C12, C12 to C13, C19 to C14, C3 to C2, C1 to C3, C20 to C4, C4 to C5, C8 to C7, C10 to C8, C5 to C9, D8 to D1, D7 to D2, D1 to D3, D2 to D4, D3 to D5, D4 to D6, D5 to D7, D6 to D8, J2 to J1, J1 to J2, P4 to P1, P1 to P2, P2 to P3, P3 to P4, R2 to R1, R9 to R10, R8 to R11, R11 to R12, R12 to R13, R20 to R14, R6 to R15, R19 to R16, R10 to R17, R13 to R18, R14 to R19, R3 to R2, R15 to R20, R24 to R21, R16 to R22, R17 to R23, R18 to R24, R4 to R3, R1 to R4, R21 to R5, R22 to R6, R23 to R7, R5 to R8, R7 to R9, U3 to U2, U2 to U3

Commit message: update broken library
Parts:
- J2: symbol dk_Rectangular-Connectors-Headers-Male-Pins:S2B-PH-SM4-TB_LF__SN_ -> Bike-Light:S2B-PH-SM4-TB_LF_SN
Changed lines of the file:
@@
 	1000 4550 1150 4550
 $Comp
-L dk_Rectangular-Connectors-Headers-Male-Pins:S2B-PH-SM4-TB_LF__SN_ J2
+L Bike-Light:S2B-PH-SM4-TB_LF_SN J2
 U 1 1 5E755FBD
 P 900 4550

Commit message: v2
Parts:
- removed J1: USB_B_Micro, bike-light-board:MICRO-USB-SMD_5PIN-H-FEMALE-PITCH0.65-L_MICRO5.9MMUSB, symbol Connector:USB_B_Micro
- added J1: USB_Micro_MICRO_4P_DIP, footprints:USB_Micro-MICRO_4P_DIP, symbol cb_Connector:USB_Micro_MICRO_4P_DIP
- C1, C12, C7: JCLPCB Part Number (none) -> C57112
- C10, C5, C9: JCLPCB Part Number (none) -> C52923
- C11, C13, C4, C6, C8: JCLPCB Part Number (none) -> C1525
- C14, C2, C3: JCLPCB Part Number (none) -> C19702
- D1: JCLPCB Part Number (none) -> C355236
- D2: JCLPCB Part Number (none) -> C2480
- F1: JCLPCB Part Number (none) -> C261937
- Q1, Q2, Q3: JCLPCB Part Number (none) -> C216792
- R1, R10, R11, R12, R13, R16, R5, R7, R8: JCLPCB Part Number (none) -> C25792
- R14, R17, R18, R2, R24, R4, R6: JCLPCB Part Number (none) -> C25744
- R15, R22, R23: JCLPCB Part Number (none) -> C25133
- R19, R20, R21, R3: JCLPCB Part Number (none) -> C25867
- R9: JCLPCB Part Number (none) -> C25790
- U1: JCLPCB Part Number (none) -> C32574
- U2: JCLPCB Part Number (none) -> C457290
- U3: JCLPCB Part Number (none) -> C277882
- U5: JCLPCB Part Number (none) -> C12493

Commit message: update to esp32-s2
Parts:
- removed C10, C9: 1u, Capacitor_SMD:C_0402_1005Metric, symbol Device:C
- removed C11: 100n, Capacitor_SMD:C_0402_1005Metric, symbol Device:C
- removed C12: 10n, Capacitor_SMD:C_0603_1608Metric, symbol Device:C
- removed J3: AVR-ISP-6, Connector_PinHeader_2.54mm:PinHeader_2x03_P2.54mm_Vertical_SMD, symbol Connector:AVR-ISP-6
- removed unit 1 of Q1
- removed R17, R6: 10k, Resistor_SMD:R_0402_1005Metric, symbol Device:R
- removed R19, R20, R21, R3: 1k5, Resistor_SMD:R_0402_1005Metric, symbol Device:R
- removed R22, R23: 68, Resistor_SMD:R_0402_1005Metric, symbol Device:R
- removed R7: 47k, Resistor_SMD:R_0402_1005Metric, symbol Device:R
- removed U2: QMA7981, Package_LGA:LGA-12_2x2mm_P0.5mm, symbol Bike-Light:QMA7981
- removed U3: SSP6206-33NR, Package_TO_SOT_SMD:SOT-23, symbol Bike-Light:SSP6206-33NR
- removed U4: ATtiny84A-MU, Package_DFN_QFN:QFN-20-1EP_4x4mm_P0.5mm_EP2.6x2.6mm, symbol MCU_Microchip_ATtiny:ATtiny84A-MU
- removed U5: M74VHC1GT08DFT2G, Package_TO_SOT_SMD:SOT-353_SC-70-5, symbol Bike-Light:M74VHC1GT08DFT2G
- added A?: ANT3216LL00R2400A, footprints:Antenna_3216, symbol cb_Antenna:ANT3216LL00R2400A
- added C? (x9): 100n, Capacitor_SMD:C_0402_1005Metric, symbol Device:C
- added C? (x3): 10u, Capacitor_SMD:C_0603_1608Metric, symbol Device:C
- added C? (x2): C_0402_50V_COG_2p2, Capacitor_SMD:C_0402_1005Metric, symbol cb_Capacitors-Ceramic:C_0402_50V_COG_2p2
- added C? (x4): 1u, Capacitor_SMD:C_0402_1005Metric, symbol Device:C
- added C? (x2): C_0402_50V_COG_20p, Capacitor_SMD:C_0402_1005Metric, symbol cb_Capacitors-Ceramic:C_0402_50V_COG_20p
- added C? (x2): DNP, Capacitor_SMD:C_0402_1005Metric, symbol cb_Capacitors-Ceramic:C_0402_50V_COG_2p2
- added L? (x2): HQ1005C2N0ST, Inductor_SMD:L_0402_1005Metric, symbol cb_Inductors:HQ1005C2N0ST
- added P?: TC2030-IDC-NL_ESP, Connector:Tag-Connect_TC2030-IDC-NL_2x03_P1.27mm_Vertical, symbol cb_Connector:TC2030-IDC-NL_ESP
- added R? (x3): 10k, Resistor_SMD:R_0402_1005Metric, symbol Device:R
- added R? (x2): 47k, Resistor_SMD:R_0402_1005Metric, symbol Device:R
- added R? (x9): 0R, symbol Device:R
- added U2: QMA7981, Package_LGA:LGA-12_2x2mm_P0.5mm, symbol cb_ICs_Sensor:QMA7981
- added U6: M74VHC1GT126DF1G, Package_TO_SOT_SMD:SOT-353_SC-70-5, symbol cb_ICs_Logic:M74VHC1GT126DF1G
- added U? (x2): ESP32-S2, Package_DFN_QFN:QFN-56-1EP_7x7mm_P0.4mm_EP5.6x5.6mm, symbol cb_ICs_Micros:ESP32-S2
- added U?: ME6231A33PG, Package_TO_SOT_SMD:SOT-89-3, symbol cb_ICs_Power:ME6231A33PG
- added U?: P25Q40H-SSH-IT, Package_SO:SOIC-8_3.9x4.9mm_P1.27mm, symbol cb_ICs_Memory:P25Q40H-SSH-IT
- added Y?: X322540MPB4SI, Crystal:Crystal_SMD_3225-4Pin_3.2x2.5mm, symbol cb_Crystals:X322540MPB4SI
Connections:
- net labels added: BT, LIGHT_SENS_EN, RF_ANT, RF_LNA, RX, SPI_FL_CLK, SPI_FL_CS, SPI_FL_D, SPI_FL_HD, SPI_FL_Q, SPI_FL_WP, TX, VBUS_MONITOR, VDD_SPI, nRESET
- net labels removed: PA0, PA1, PA2, PA3, PA4, PA5, PA6, PA7, PB0, PB1, PB2, PROG_CLK, PROG_MISO, PROG_MOSI, PROG_nRESET, RESET, VBUS_FET_EN
- wire segments 196 -> 255
- no-connect marks 7 -> 10
Other:
- note added: "4M external flash"
- note added: "C = 2 * ( CL - Cstray )\nC = 2 * ( 15p - 5p )"
- note added: "If RTC crystal is not required\ncan use 21 and 22 as IO pins"
- note added: "Matching circuit should be tuned\nbased on PCB layout"
- note added: "Place near\nchip"
- note added: "Pullup on U1RX\nto avoid boot issues"
- note added: "RC delays startup\nSuggested 1u 10k"
- note added: "Seperate from LED power since when plugged in want to measure battery and not VLED"
- note added: "Series resistors to reduce\ninterference to wifi, ajust if needed"
- moved on the sheet: C1, C13, C2, C3, C4, C5, C6, C7, J2, R1, R18, R24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

Commit message: more updates
Parts:
- removed Q1, Q2, Q3: NCE2003, Package_TO_SOT_SMD:SOT-23-6, symbol Bike-Light:NCE2003
- removed R15: 68, Resistor_SMD:R_0402_1005Metric, symbol Device:R
- added Q1, Q3, Q5: HX2301A, Package_TO_SOT_SMD:SOT-23, symbol cb_Transistors-FETs:HX2301A
- added Q2: L2N7002DW1T1G, Package_TO_SOT_SMD:SOT-363_SC-70-6, symbol cb_Transistors-FETs:L2N7002DW1T1G
- R14: value 10k -> 47k; JCLPCB Part Number C25744 -> (none); LCSC Part Number C60490 -> (none)
- R17, R19, R20, R21, R25, R26, R27, R6, R7: renamed from R?; footprint (none) -> Resistor_SMD:R_0402_1005Metric
- gave numbers to parts that had none: 35
Connections:
- net +BATT: now also Q1.3 (D), Q3.2 (S)
- net +VSW: now also Q5.3 (D)
- net GND: now also Q2.1 (S), Q2.4 (S)
- net SW_EN: now also Q2.2 (G), Q2.5 (G)
- net USB_D+: now also R25.1, U3.26 (D+/GPIO20); no longer C29.1, D1.1 (K), J1.3 (D+), R26.2
- net USB_D-: now also R26.1, U3.25 (D-/GPIO19); no longer C28.1, D1.4 (K), J1.2 (D-), R25.2
- net VSUP: now also Q1.2 (S), Q5.2 (S)
- net at R8.1: now also Q1.1 (G)
- net at R11.2: now also Q2.6 (D)
- net at R11.1, R9.2: now also Q5.1 (G)
- net at R10.2: now also Q2.3 (D), Q3.1 (G)
- net at R12.1: now also Q3.3 (D)
- new net: C28.1, D1.1 (K), J1.3 (D+), R25.2
- new net: C29.1, D1.4 (K), J1.2 (D-), R26.2
- no-connect marks 10 -> 9
Other:
- note added: "TODO check pinout"
- moved on the sheet: C28, C29, C30, C31, C32, D2, Q4, R11, R16, R25, R26, R28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

Commit message: clean up schematic
Parts:
- removed C4: 100n, Capacitor_SMD:C_0402_1005Metric, symbol Device:C
- removed P1, P4: WirePad, bike-light-board:Solder_Wire_Pad_5mmx3mm, symbol Bike-Light:WirePad
- added TP1, TP10, TP11, TP12, TP13, TP14, TP16, TP17, TP18, TP19, TP2, TP3, TP4, TP5, TP6, TP7, TP8, TP9: TestPoint_ICT_1mm, footprints:ICT_TestPoint_Pad_D1.00mm, symbol cb_Test-Points:TestPoint_ICT_1mm
Connections:
- net +3V3: now also P5.2 (VDD), TP19.1; no longer P5.1 (EN)
- net +VSW: now also TP18.1
- net BT: no longer P5.4 (GND)
- net CHRG_STAT: now also TP13.1
- net GND: now also P5.4 (GND), TP5.1; no longer P5.6 (IO0)
- net RX: now also TP11.1
- net TX: now also TP10.1
- net VBUS: now also R8.1; no longer R8.2
- net VSUP: now also TP17.1
- net nRESET: no longer P5.2 (VDD)
- net at C1.1, R1.1, R2.2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: now also TP8.1
- net at C28.1, D1.1 (K), J1.3 (D+)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: now also TP6.1
- net at C29.1, D1.4 (K), J1.2 (D-)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: now also TP7.1
- net at D1.5 (K), F1.2, J1.1 (VBUS): now also TP9.1
- net CHRG_I_MONITOR: now reaches R4.1, U1.5 (PROG)
- net CHRG_I_MONITOR: now also U3.13 (GPIO8)
- net at Q1.1 (G): now also R8.2; no longer R8.1
- net at U3.43 (MTCK/JTAG/GPIO39): now also TP1.1
- net at U3.44 (MTDO/JTAG/GPIO40): now also TP2.1
- net at U3.46 (MTDI/JTAG/GPIO41): now also TP3.1
- net at U3.47 (MTMS/JTAG/GPIO42): now also TP4.1
- net +BATT renamed VBAT
- net VBAT: now also TP16.1
- net BATT_MONITOR renamed VBAT_MONITOR
- new net EN: P5.1 (EN), TP12.1
- new net IO0: P5.6 (IO0), TP14.1
Other:
- note added: "3.3V"
- note added: "BAT / USB POWER SELECT"
- note added: "BATTERY CHARGER"
- note added: "BUTTON"
- note added: "Divider is switched off\nto save battery"
- note added: "ESP32-S2 IO"
- note added: "ESP32-S2 POWER"
- note added: "Icharge = 1000/R4\nIcharge = 100 mA"
- note added: "LEDS"
- note added: "LIGHT SENSOR"
- note added: "Level shifter\n3V3 logic to 5V LED logic"
- note added: "MOTION SENSOR"
- note added: "SWITCHED LED POWER"
- note added: "To save battery\nwhen LEDs are off"
- note added: "USB"
- note added: "Used to detect USB connected"
- note removed: "3.3V Regulator"
- note removed: "Accelerometer"
- note removed: "Battery Charger"
- note removed: "Battery Connector"
- note removed: "Button"
- note removed: "Icharge = 1000/R1\nIcharge = 100 mA"
- note removed: "LED Switched Power"
- note removed: "LEDs"
- note removed: "Light Sensor"
- note removed: "Microcontroller"
- note removed: "Seperate from LED power since when plugged in want to measure battery and not VLED"
- note removed: "Switched Battery Monitor"
- note removed: "TODO check pinout"
- note removed: "USB Connector"
- note removed: "USB/ Battery Power Select"
- moved on the sheet: A1, C1, C10, C11, C12, C13, C14, C15, C16, C17, C18, C19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

Commit message: placement
Parts:
- removed J1: USB_Micro_MICRO_4P_DIP, footprints:USB_Micro-MICRO_4P_DIP, symbol cb_Connector:USB_Micro_MICRO_4P_DIP
- removed P5: TC2030-IDC-NL_ESP, Connector:Tag-Connect_TC2030-IDC-NL_2x03_P1.27mm_Vertical, symbol cb_Connector:TC2030-IDC-NL_ESP
- removed R21: 0R, Resistor_SMD:R_0402_1005Metric, symbol Device:R
- removed TP1, TP16, TP2, TP3, TP4: TestPoint_ICT_1mm, footprints:ICT_TestPoint_Pad_D1.00mm, symbol cb_Test-Points:TestPoint_ICT_1mm
- added C33: 10n, Capacitor_SMD:C_0603_1608Metric, symbol Device:C
- added C4: 100n, Capacitor_SMD:C_0402_1005Metric, symbol Device:C
- added J1: KH-TYPE-C-16P, footprints:USB_C_Receptacle_KH-TYPE-C-16P, symbol cb_Connector:KH-TYPE-C-16P
- added R15: 2k, Resistor_SMD:R_0402_1005Metric, symbol Device:R
- added SW2, SW3: STO-060A16AB, footprints:STO-060A16AB, symbol cb_Switch:STO-060A16AB
- C12: value 1u -> 10n; footprint Capacitor_SMD:C_0402_1005Metric -> Capacitor_SMD:C_0603_1608Metric; Derating (none) -> X7R; JCLPCB Part Number C52923 -> C57112; LCSC Part Number C497333 -> C77439; Voltage (none) -> 100
- R17: value 0R -> 2k; JCLPCB Part Number (none) -> C25744; LCSC Part Number (none) -> C60490
- R19, R20: value 0R -> 5k1
- R22: value 10k -> DNP; JCLPCB Part Number C25744 -> (none); LCSC Part Number C60490 -> (none)
- U3: footprint Package_DFN_QFN:QFN-56-1EP_7x7mm_P0.4mm_EP5.6x5.6mm -> footprints:ESP32-S2
Connections:
- net BT is gone; now on net IO0: U3.5 (GPIO0/STRAP)
- net nRESET is gone; now on net EN: C21.1, R3.1, U3.56 (CHIP/PU/RESET)
- net +3V3: now also C4.1; no longer C12.1
- net ACCEL_INT: now also U3.10 (GPIO5); no longer U3.11 (GPIO6)
- net BUTTON: now also U3.23 (DAC_1/GPIO18); no longer U3.10 (GPIO5)
- net CHRG_I_MONITOR: now also U3.15 (GPIO10); no longer U3.13 (GPIO8)
- net CHRG_STAT: now also U3.14 (GPIO9); no longer U3.9 (GPIO4)
- net EN: now also R17.2; no longer TP12.1
- net GND: now also R19.2, R20.2, C33.2, C4.2, J1.A1 (GND), J1.A12 (GND), J1.B1 (GND), J1.B12 (GND), SW2.1, SW3.1
- net IO0: now also R15.2; no longer TP14.1
- net LED_DATA: now also U3.16 (GPIO11); no longer U3.39 (GPIO35)
- net LIGHT_SENS: now also U3.13 (GPIO8); no longer U3.8 (GPIO3)
- net LIGHT_SENS_EN: now also U3.41 (GPIO37); no longer U3.12 (GPIO7)
- net SPI_FL_CLK: now also R7.2; no longer R19.1
- net SPI_FL_D: now also U3.36 (SPID/GPIO32)
- net SPI_FL_HD: now also U3.31 (SPIHD/GPIO27); no longer R17.1
- net SPI_FL_Q: now also U3.35 (SPIQ/GPIO31); no longer R20.1
- net SPI_FL_WP: now also U3.32 (SPIWP/GPIO28); no longer R7.1
- net SW_EN: now also U3.42 (GPIO38); no longer U3.41 (GPIO37)
- net VBAT_MONITOR: now also U3.12 (GPIO7); no longer U3.7 (GPIO2)
- net VBUS_MONITOR: now also U3.11 (GPIO6); no longer U3.6 (GPIO1)
- net USB+: now reaches C28.1, R25.2, TP6.1
- net USB+: now also D1.5 (K), J1.A6 (D+), J1.B6 (D+); no longer D1.1 (K)
- net VBUS_IN: now reaches D1.3 (K)
- net VBUS_IN: now also F1.2, TP9.1, J1.A4 (VBUS), J1.A9 (VBUS), J1.B4 (VBUS), J1.B9 (VBUS)
- net USB-: now reaches C29.1, D1.4 (K), R26.2, TP7.1
- net USB-: now also J1.A7 (D-), J1.B7 (D-)
- net at R23.1: now also U3.24 (DAC_2/GPIO17); no longer U3.23 (DAC_1/GPIO18)
- net MTCK: now reaches U3.43 (MTCK/JTAG/GPIO39)
- net MTDO: now reaches U3.44 (MTDO/JTAG/GPIO40)
- net MTDI: now reaches U3.46 (MTDI/JTAG/GPIO41)
- net MTMS: now reaches U3.47 (MTMS/JTAG/GPIO42)
- net at U3.34 (SPICLK/GPIO30): now also R7.1; no longer R19.2
- new net: J1.A5 (CC1), R20.1
- new net: J1.B5 (CC2), R19.1
- new net: C12.1, R15.1, SW2.2, TP14.1
- new net: C33.1, R17.1, SW3.2, TP12.1
- no-connect marks 9 -> 10
Other:
- note added: "OPTIONAL EN, BOOT BUTTON"
- note added: "Place each cap\nnear respective pin"
- note removed: "Series resistors to reduce\ninterference to wifi, ajust if needed"
- moved on the sheet: C1, C2, C28, C29, C3, C30, C31, C32, C8, D1, D2, F1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
