File: bike-light-board.sch (KiCad schematic (older format))
At the start: 105 parts, among them J1 KH-TYPE-C-16P, J2 S2B-PH-SM4-TB, P2 WirePad, P3 WirePad, Q1 HX2301A, Q2 L2N7002DW1T1G, Q3 HX2301A, Q4 SMD0805-20, Q5 HX2301A, SW1 SW_Push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

Commit message: routing done
Parts:
- removed TP13: TestPoint_ICT_1mm, footprints:ICT_TestPoint_Pad_D1.00mm, symbol cb_Test-Points:TestPoint_ICT_1mm
Connections:
- net BUTTON: now also U3.23 (DAC_1/GPIO17); no longer U3.24 (DAC_2/GPIO18)
- net at R23.1: now also U3.24 (DAC_2/GPIO18); no longer U3.23 (DAC_1/GPIO17)
Other:
- moved on the sheet: R23
Changed lines of the file:
@@
 L Device:R R23
 U 1 1 612F8DF5
-P 8800 7650
-F 0 "R23" H 8870 7696 50  0000 L CNN
-F 1 "10k" H 8870 7605 50  0000 L CNN
-F 2 "Resistor_SMD:R_0402_1005Metric" V 8730 7650 50  0001 C CNN
-F 3 "~" H 8800 7650 50  0001 C CNN
-F 4 "C60490" H 8800 7650 50  0001 C CNN "LCSC Part Number"
-F 5 "C25744" H 8800 7650 50  0001 C CNN "JCLPCB Part Number"
-	1    8800 7650
+P 8800 7750
+F 0 "R23" H 8870 7796 50  0000 L CNN
+F 1 "10k" H 8870 7705 50  0000 L CNN
+F 2 "Resistor_SMD:R_0402_1005Metric" V 8730 7750 50  0001 C CNN
+F 3 "~" H 8800 7750 50  0001 C CNN
+F 4 "C60490" H 8800 7750 50  0001 C CNN "LCSC Part Number"
+F 5 "C25744" H 8800 7750 50  0001 C CNN "JCLPCB Part Number"
+	1    8800 7750
 	1    0    0    1
 $EndComp
@@
 L power:+3.3V #PWR0130
 U 1 1 6130F896
-P 8800 7500
-F 0 "#PWR0130" H 8800 7350 50  0001 C CNN
-F 1 "+3.3V" H 8815 7673 50  0000 C CNN
-F 2 "" H 8800 7500 50  0001 C CNN
-F 3 "" H 8800 7500 50  0001 C CNN
-	1    8800 7500
-	1    0    0    -1
-$EndComp
-Wire Wire Line
-	8800 7800 8800 7850
-Text Notes 8250 8050 0    50   Italic 0
+P 8800 7600
+F 0 "#PWR0130" H 8800 7450 50  0001 C CNN
+F 1 "+3.3V" H 8815 7773 50  0000 C CNN
+F 2 "" H 8800 7600 50  0001 C CNN
+F 3 "" H 8800 7600 50  0001 C CNN
+	1    8800 7600
+	1    0    0    -1
+$EndComp
+Wire Wire Line
+	8800 7900 8800 7950
+Text Notes 8350 8150 0    50   Italic 0
 Pullup on U1RX\nto avoid boot issues
 $Comp
@@
 Text GLabel 9750 7250 0    50   Input ~ 0
 CHRG_STAT
-Text GLabel 9750 7950 0    50   Input ~ 0
+Text GLabel 9750 7850 0    50   Input ~ 0
 BUTTON
 Text GLabel 9750 7050 0    50   Input ~ 0
@@
 	9950 6850 9750 6850
 Wire Wire Line
-	9950 7950 9750 7950
+	9950 7850 9750 7850
 Wire Wire Line
 	9950 7250 9750 7250
@@
 Wire Wire Line
 	4850 2900 4600 2900
-Wire Wire Line
-	5100 2900 5000 2900
 Connection ~ 4850 2900
-$Comp
-L cb_Test-Points:TestPoint_ICT_1mm TP13
-U 1 1 61B9D273
-P 5000 2900
-F 0 "TP13" H 5000 2975 50  0001 C CNN
-F 1 "TestPoint_ICT_1mm" H 5000 2980 50  0001 C CNN
-F 2 "footprints:ICT_TestPoint_Pad_D1.00mm" H 5200 2900 50  0001 C CNN
-F 3 "~" H 5200 2900 50  0001 C CNN
-	1    5000 2900
-	1    0    0    -1
-$EndComp
-Connection ~ 5000 2900
-Wire Wire Line
-	5000 2900 4850 2900
 Connection ~ 4400 1100
 Wire Wire Line
@@
 VBUS_IN
 Wire Wire Line
-	8800 7850 9950 7850
+	8800 7950 9950 7950
 Wire Wire Line
 	2750 2900 3550 2900
@@
 Wire Wire Line
 	2150 2150 2150 2350
+Wire Wire Line
+	4850 2900 5100 2900
 $EndSCHEMATC

Commit message: Update BOM
Parts:
- A1: JCLPCB Part Number (none) -> C293767
- C16, C17: JCLPCB Part Number (none) -> C1554
- C24, C26: JCLPCB Part Number (none) -> C1559
- J1: JCLPCB Part Number (none) -> C709357
- L1, L2: JCLPCB Part Number (none) -> C145023
- Q1, Q3, Q5: JCLPCB Part Number (none) -> C10487
- Q2: JCLPCB Part Number (none) -> C61840
- R14: JCLPCB Part Number (none) -> C25792
- R15, R17: JCLPCB Part Number C25744 -> C4109
- R19, R20: JCLPCB Part Number (none) -> C25905
- R25, R26, R27, R6, R7: JCLPCB Part Number (none) -> C17168
- SW1: JCLPCB Part Number (none) -> C10852
- U3: JCLPCB Part Number (none) -> C529594
- U4: JCLPCB Part Number (none) -> C194873
- U5: JCLPCB Part Number (none) -> C2681684
- Y1: JCLPCB Part Number (none) -> C9010
Changed lines of the file:
@@
 F 3 "~" H 13150 6750 50  0001 C CNN
 F 4 "C412370" H 13150 6550 50  0001 C CNN "LCSC Part Number"
+F 5 "C10852" H 13150 6550 50  0001 C CNN "JCLPCB Part Number"
 	1    13150 6550
 	0    -1   1    0
@@
 F 4 "0402" H 6100 3700 50  0001 C CNN "Package Size"
 F 5 "1%" H 6100 3700 50  0001 C CNN "Tolerance"
+F 6 "C25792" H 6100 3700 50  0001 C CNN "JCLPCB Part Number"
 	1    6100 3700
 	1    0    0    -1
@@
 F 3 "~" H 2550 6900 50  0001 C CNN
 F 4 "2nH" V 2450 6900 50  0000 C CNN "Inductance"
+F 5 "C145023" H 2550 6900 50  0001 C CNN "JCLPCB Part Number"
 	1    2550 6900
 	0    -1   -1   0
@@
 F 2 "Package_SO:SOIC-8_3.9x4.9mm_P1.27mm" H 7150 7700 50  0001 C CNN
 F 3 "https://www.adestotech.com/wp-content/uploads/DS-AT25SF081_045.pdf" H 7150 8300 50  0001 C CNN
+F 4 "C194873	" H 7150 8300 50  0001 C CNN "JCLPCB Part Number"
 	1    7150 8300
 	1    0    0    -1
@@
 F 5 "COG/NPO" H 2700 8950 50  0001 C CNN "Derating"
 F 6 "20p" V 2800 9100 50  0000 C CNN "Capacitance"
+F 7 "C1554" H 2700 8950 50  0001 C CNN "JCLPCB Part Number"
 	1    2700 8950
 	0    1    1    0
@@
 F 5 "COG/NPO" H 2700 8550 50  0001 C CNN "Derating"
 F 6 "20p" V 2600 8700 50  0000 C CNN "Capacitance"
+F 7 "C1554" H 2700 8550 50  0001 C CNN "JCLPCB Part Number"
 	1    2700 8550
 	0    1    1    0
@@
 F 3 "~" H 2900 8750 50  0001 C CNN
 F 4 "40MHz" V 3150 8800 50  0000 L CNN "Frequency"
+F 5 "C9010" H 2900 8750 50  0001 C CNN "JCLPCB Part Number"
 	1    2900 8750
 	0    1    1    0
@@
 F 2 "Resistor_SMD:R_0402_1005Metric" V 3080 8550 50  0001 C CNN
 F 3 "~" H 3150 8550 50  0001 C CNN
+F 4 "C17168" H 3150 8550 50  0001 C CNN "JCLPCB Part Number"
 	1    3150 8550
 	0    -1   -1   0
@@
 F 2 "footprints:Antenna_3216" H 6550 9450 50  0001 C CNN
 F 3 "https://www.yageo.com/upload/media/product/productsearch/datasheet/wireless/An_Ceramiz_2450_3216_L00_0.pdf" H 6550 9450 50  0001 C CNN
+F 4 "C293767	" H 6800 9250 50  0001 C CNN "JCLPCB Part Number"
 	1    6800 9250
 	1    0    0    -1
@@
 F 3 "~" H 6000 9450 50  0001 C CNN
 F 4 "2nH" V 5900 9450 50  0000 C CNN "Inductance"
+F 5 "C145023" H 6000 9450 50  0001 C CNN "JCLPCB Part Number"
 	1    6000 9450
 	0    -1   -1   0
@@
 F 5 "COG/NPO" H 6300 9650 50  0001 C CNN "Derating"
 F 6 "2p2" H 6392 9559 50  0000 L CNN "Capacitance"
+F 7 "C1559" H 6300 9650 50  0001 C CNN "JCLPCB Part Number"
 	1    6300 9650
 	1    0    0    -1
@@
 F 5 "COG/NPO" H 5650 9650 50  0001 C CNN "Derating"
 F 6 "2p2" H 5742 9559 50  0000 L CNN "Capacitance"
+F 7 "C1559" H 5650 9650 50  0001 C CNN "JCLPCB Part Number"
 	1    5650 9650
 	1    0    0    -1
@@
 F 2 "footprints:ESP32-S2" H 15000 6950 50  0001 C CNN
 F 3 "https://www.espressif.com/sites/default/files/documentation/esp32-s2_datasheet_en.pdf" H 10350 8100 50  0001 C CNN
+F 4 "C529594" H 10950 7650 50  0001 C CNN "JCLPCB Part Number"
 	1    10950 7650
 	1    0    0    -1
@@
 F 2 "Package_TO_SOT_SMD:SOT-89-3" H 7300 1575 50  0001 C CIN
 F 3 "https://datasheet.lcsc.com/lcsc/2101201002_MICRONE-Nanjing-Micro-One-Elec-ME6231A33PG_C2681684.pdf" H 7300 1350 50  0001 C CNN
+F 4 "C2681684" H 7300 1350 50  0001 C CNN "JCLPCB Part Number"
 	1    7300 1350
 	1    0    0    -1
@@
 F 2 "Resistor_SMD:R_0402_1005Metric" V 9480 9350 50  0001 C CNN
 F 3 "~" H 9550 9350 50  0001 C CNN
+F 4 "C17168" H 9550 9350 50  0001 C CNN "JCLPCB Part Number"
 	1    9550 9350
 	0    1    1    0
@@
 F 2 "Resistor_SMD:R_0402_1005Metric" V 3480 1300 50  0001 C CNN
 F 3 "~" H 3550 1300 50  0001 C CNN
+F 4 "C17168" H 3550 1300 50  0001 C CNN "JCLPCB Part Number"
 	1    3550 1300
 	0    1    1    0
@@
 F 2 "Package_TO_SOT_SMD:SOT-23" H 5450 1750 50  0001 C CNN
 F 3 "https://datasheet.lcsc.com/szlcsc/1912111437_HX-hengjiaxing-HX2301A_C296298.pdf" H 5250 1650 50  0001 C CNN
+F 4 "C10487" H 5250 1650 50  0001 C CNN "JCLPCB Part Number"
 	1    5250 1650
 	0    -1   1    0
@@
 F 2 "Package_TO_SOT_SMD:SOT-363_SC-70-6" H 7300 4950 50  0001 C CNN
 F 3 "https://datasheet.lcsc.com/lcsc/1912111437_LRC-L2N7002DW1T1G_C383161.pdf" H 7300 4950 50  0001 C CNN
+F 4 "C61840" H 7100 4950 50  0001 C CNN "JCLPCB Part Number"
 	2    7100 4950
 	1    0    0    -1
@@
 F 2 "Package_TO_SOT_SMD:SOT-23" H 7400 4550 50  0001 C CNN
 F 3 "https://datasheet.lcsc.com/szlcsc/1912111437_HX-hengjiaxing-HX2301A_C296298.pdf" H 7200 4450 50  0001 C CNN
+F 4 "C10487" H 7200 4450 50  0001 C CNN "JCLPCB Part Number"
 	1    7200 4450
 	0    1    -1   0
@@
 F 2 "footprints:ESP32-S2" H 5600 5850 50  0001 C CNN
 F 3 "https://www.espressif.com/sites/default/files/documentation/esp32-s2_datasheet_en.pdf" H 3750 8100 50  0001 C CNN
+F 4 "C529594" H 4350 7650 50  0001 C CNN "JCLPCB Part Number"
 	2    4350 7650
 	1    0    0    -1
@@
 F 2 "Package_TO_SOT_SMD:SOT-363_SC-70-6" H 7300 3450 50  0001 C CNN
 F 3 "https://datasheet.lcsc.com/lcsc/1912111437_LRC-L2N7002DW1T1G_C383161.pdf" H 7300 3450 50  0001 C CNN
+F 4 "C61840" H 7100 3450 50  0001 C CNN "JCLPCB Part Number"
 	1    7100 3450
 	1    0    0    -1
@@
 F 2 "Package_TO_SOT_SMD:SOT-23" H 7400 2750 50  0001 C CNN
 F 3 "https://datasheet.lcsc.com/szlcsc/1912111437_HX-hengjiaxing-HX2301A_C296298.pdf" H 7200 2650 50  0001 C CNN
+F 4 "C10487" H 7200 2650 50  0001 C CNN "JCLPCB Part Number"
 	1    7200 2650
 	0    1    -1   0
@@
 F 2 "Resistor_SMD:R_0402_1005Metric" V 5530 8450 50  0001 C CNN
 F 3 "~" H 5600 8450 50  0001 C CNN
+F 4 "C17168" H 5600 8450 50  0001 C CNN "JCLPCB Part Number"
 	1    5600 8450
 	0    -1   -1   0
@@
 F 3 "~" H 12950 8250 50  0001 C CNN
 F 4 "C60490" H 12950 8250 50  0001 C CNN "LCSC Part Number"
-F 5 "C25744" H 12950 8250 50  0001 C CNN "JCLPCB Part Number"
+F 5 "C4109" H 12950 8250 50  0001 C CNN "JCLPCB Part Number"
 	1    12950 8250
 	0    1    -1   0
@@
 F 3 "~" H 14450 8250 50  0001 C CNN
 F 4 "C60490" H 14450 8250 50  0001 C CNN "LCSC Part Number"
-F 5 "C25744" H 14450 8250 50  0001 C CNN "JCLPCB Part Number"
+F 5 "C4109" H 14450 8250 50  0001 C CNN "JCLPCB Part Number"
 	1    14450 8250
 	0    1    -1   0
@@
 F 3 "https://datasheet.lcsc.com/lcsc/2009111434_Shenzhen-Kinghelm-Elec-KH-TYPE-C-16P_C709357.pdf" H 1250 1700 50  0001 C CNN
 F 4 "C709357" H 1100 1700 50  0001 C CNN "JCLPCB"
+F 5 "C709357" H 1100 1700 50  0001 C CNN "JCLPCB Part Number"
 	1    1100 1700
 	1    0    0    -1
@@
 F 2 "Resistor_SMD:R_0402_1005Metric" V 3480 1500 50  0001 C CNN
 F 3 "~" H 3550 1500 50  0001 C CNN
+F 4 "C17168" H 3550 1500 50  0001 C CNN "JCLPCB Part Number"
 	1    3550 1500
 	0    1    1    0
@@
 F 2 "Resistor_SMD:R_0402_1005Metric" V 1780 2500 50  0001 C CNN
 F 3 "~" H 1850 2500 50  0001 C CNN
+F 4 "C25905" H 1850 2500 50  0001 C CNN "JCLPCB Part Number"
 	1    1850 2500
 	-1   0    0    -1
@@
 F 2 "Resistor_SMD:R_0402_1005Metric" V 2080 2500 50  0001 C CNN
 F 3 "~" H 2150 2500 50  0001 C CNN
+F 4 "C25905" H 2150 2500 50  0001 C CNN "JCLPCB Part Number"
 	1    2150 2500
 	-1   0    0    -1
