File: lil-lite-board.sch (KiCad schematic (older format))
At the start: 105 parts, among them J1 KH-TYPE-C-16P, J2 S2B-PH-SM4-TB, P2 WirePad, P3 WirePad, Q1 HX2301A, Q2 L2N7002DW1T1G, Q3 HX2301A, Q4 SMD0805-20, Q5 HX2301A, SW1 TS5220A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

Commit message: Change VBUS divider for digital in
Parts:
- R28: value 10k -> 5k1; JCLPCB Part Number C25744 -> (none)
- R29: value 5k1 -> 10k; JCLPCB Part Number C25905 -> (none)
Changed lines of the file:
@@
 P 4300 4550
 F 0 "R28" H 4370 4596 50  0000 L CNN
-F 1 "10k" H 4370 4505 50  0000 L CNN
+F 1 "5k1" H 4370 4505 50  0000 L CNN
 F 2 "Resistor_SMD:R_0402_1005Metric" V 4230 4550 50  0001 C CNN
 F 3 "~" H 4300 4550 50  0001 C CNN
-F 4 "C25744" H 4300 4550 50  0001 C CNN "JCLPCB Part Number"
+F 4 "" H 4300 4550 50  0001 C CNN "JCLPCB Part Number"
 	1    4300 4550
 	1    0    0    -1
@@
 P 4300 4950
 F 0 "R29" H 4370 4996 50  0000 L CNN
-F 1 "5k1" H 4370 4905 50  0000 L CNN
+F 1 "10k" H 4370 4905 50  0000 L CNN
 F 2 "Resistor_SMD:R_0402_1005Metric" V 4230 4950 50  0001 C CNN
 F 3 "~" H 4300 4950 50  0001 C CNN
-F 4 "C25905" H 4300 4950 50  0001 C CNN "JCLPCB Part Number"
+F 4 "" H 4300 4950 50  0001 C CNN "JCLPCB Part Number"
 	1    4300 4950
 	1    0    0    -1
