File: lil-lite-board.kicad_pcb (KiCad board)
At the start: 4 copper layers, 40.2 x 69 mm, 106 parts, among them J1 KH-TYPE-C-16P, J2 S2B-PH-SM4-TB, P2 WirePad, P3 WirePad, Q1 HX2301A, Q2 L2N7002DW1T1G, Q3 HX2301A, Q4 SMD0805-20, Q5 HX2301A, SW1 TS5220A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

Commit message: remove via in pad from dfm
Routing:
- net GND: vias 79 -> 78
Changed lines of the file:
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@@
     (thickness 1.6)
     (drawings 58)
-    (tracks 952)
+    (tracks 951)
     (zones 0)
     (modules 106)
@@
   (layers
     (0 F.Cu signal)
-    (1 In1.Cu signal)
-    (2 In2.Cu signal)
+    (1 In1.Cu signal hide)
+    (2 In2.Cu signal hide)
     (31 B.Cu signal)
     (32 B.Adhes user hide)
@@
     (35 F.Paste user hide)
     (36 B.SilkS user hide)
-    (37 F.SilkS user hide)
+    (37 F.SilkS user)
     (38 B.Mask user hide)
     (39 F.Mask user hide)
@@
     (47 F.CrtYd user hide)
     (48 B.Fab user hide)
-    (49 F.Fab user hide)
+    (49 F.Fab user)
   )
   (setup
@@
   (via (at 159.7 86.37) (size 0.5) (drill 0.2) (layers F.Cu B.Cu) (net 1))
   (via (at 159.5 83.42) (size 0.5) (drill 0.2) (layers F.Cu B.Cu) (net 1))
-  (via (at 159.7 84.12) (size 0.5) (drill 0.2) (layers F.Cu B.Cu) (net 1))
   (via (at 159.5 82.12) (size 0.5) (drill 0.2) (layers F.Cu B.Cu) (net 1))
   (via (at 153 94.67) (size 0.5) (drill 0.2) (layers F.Cu B.Cu) (net 1))
